Commit message: making simple squiggle to debug - definitely a weld issue. I hate this code though so i want to refactor it

File: assets/squiggle.urdf (robot description, URDF)
Before this commit: robot squiggle, 3 links, 2 joints
Links:
- removed link link1
- removed link link2
- removed link link3
- added link link1-bone; collision box size=1 0.1 0.1
- added link link1-rotor; collision cylinder length=0.1 radius=0.1
- added link link1-stator; collision cylinder length=0.1 radius=0.1
- added link link2-bone; collision box size=1 0.1 0.1
- added link link2-rotor; collision cylinder length=0.1 radius=0.1
- added link link2-stator; collision cylinder length=0.1 radius=0.1
Joints:
- removed joint q2
- added joint link1-bone-to-stator: type fixed, parent link1-bone, child link1-stator, origin xyz=1 0 0 rpy=0 0 0
- added joint link1-rotor-to-bone: type fixed, parent link1-rotor, child link1-bone, origin xyz=0 0 0 rpy=0 0 0
- added joint link2-bone-to-stator: type fixed, parent link2-bone, child link2-stator, origin xyz=1 0 0 rpy=0 0 0
- added joint link2-rotor-to-bone: type fixed, parent link2-rotor, child link2-bone, origin xyz=0 0 0 rpy=0 0 0
- joint q1: child link2 -> link2-rotor; parent link1 -> link1-stator
