Commit message: scaling

File: assets/puppet.urdf (robot description, URDF)
Before this commit: robot puppet, 38 links, 36 joints
Joints:
- joint upper-torso-stator-to-base-rotor: type continuous -> fixed

Commit message: eye added to urdf

File: assets/puppet.urdf (robot description, URDF)
Before this commit: robot puppet, 38 links, 36 joints
Links:
- added link eye; collision cylinder length=5e-3 radius=10e-3; visual cylinder length=5e-3 radius=10e-3
- added link eye-virtual-1
- added link eye-virtual-2
- added link head; collision sphere radius=32e-3; visual sphere radius=32e-3
- link upper-torso: geometry collision cylinder length=20e-3 radius=27e-3; collision cylinder length=60e-3 radius=40e-3
Joints:
- added joint eye-pitch: type continuous, parent eye-virtual-1, child eye-virtual-2, origin xyz=0 0 0 rpy=1.57079633 0 0, axis 0 0 1
- added joint eye-stalk: type fixed, parent eye-virtual-2, child eye, origin xyz=32e-3 0 0 rpy=0 0 0, axis 0 0 1
- added joint eye-yaw: type continuous, parent head, child eye-virtual-1, origin xyz=0 0 0 rpy=0 0 0, axis 0 0 1
- added joint neck-virtual: type fixed, parent upper-torso, child head, origin xyz=0 0 23e-3 rpy=0 0 0, axis 0 0 1

Commit message: upgraded dynamic robot with index based accessor, updated encoder manager to expect 10 encoders

File: assets/puppet.urdf (robot description, URDF)
Before this commit: robot puppet, 42 links, 40 joints
Links:
- link eye-virtual-1: geometry collision cylinder length=1e-3 radius=1e-3
- link eye-virtual-2: geometry collision cylinder length=1e-3 radius=1e-3
Joints:
- joint link1-bone-to-stator-left: origin xyz=0 37.5e-3 0 rpy=1.57079633 0 0 -> xyz=0 0 -42.0e-3 rpy=0 -1.57079633 0
- joint link1-bone-to-stator-right: origin xyz=0 -37.5e-3 0 rpy=-1.57079633 0 0 -> xyz=0 0 -42.0e-3 rpy=0 -1.57079633 0
- joint link2-bone-to-stator-left: origin xyz=-40e-3 0 0 rpy=0 1.57079633 0 -> xyz=0 -40e-3 0 rpy=-1.57079633 1.57079633 0
- joint link2-bone-to-stator-right: origin xyz=-40e-3 0 0 rpy=0 1.57079633 0 -> xyz=0 40e-3 0 rpy=1.57079633 1.57079633 0
- joint link3-bone-to-stator-left: origin xyz=0 -20e-3 -45e-3 rpy=0 1.57079633 3.14159265359 -> xyz=20e-3 0 -45e-3 rpy=1.57079633 1.57079633 3.14159265359
- joint link3-bone-to-stator-right: origin xyz=0 20e-3 -45e-3 rpy=0 1.57079633 3.14159265359 -> xyz=20e-3 0 -45e-3 rpy=-1.57079633 1.57079633 3.14159265359
- joint uppertorso-bone-upperarmstator: origin xyz=0 -40e-3 0 rpy=0 -1.57079633 0 -> xyz=0 -30e-3 0 rpy=-1.57079633 0 0

Commit message: remove eye, try pd servoing law, stable

File: assets/puppet.urdf (robot description, URDF)
Before this commit: robot puppet, 42 links, 40 joints
Links:
- removed link eye
- removed link eye-virtual-1
- removed link eye-virtual-2
Joints:
- removed joint eye-pitch
- removed joint eye-stalk
- removed joint eye-yaw
